Commit message: reconstracted hole model

File: urdf/circle_10mm.urdf (robot description, URDF)
Before this commit: robot insertion_box.urdf, 2 links, 1 joints
Links:
- link box: geometry collision mesh filename=stl/collision/circle_10mm.STL scale=0.002 0.002 0.002; visual mesh filename=stl/visual/circle_10mm.STL scale=0.002 0.002 0.002
