Commit message: add peg in hole env

File: urdf/pipe.urdf (robot description, URDF)
Before this commit: robot pipe, 25 links, 24 joints
Links:
- removed link pipe_link1100.11
- added link pipe_link10.0111, mass 0.0111; collision mesh filename=../obj/cylinder_3_1_1.obj; visual mesh filename=../obj/cylinder_3_1_1.obj
- link pipe_link0: mass 100.11 -> 0.00111
- link pipe_link1: mass 100.11 -> 0.0111
- link pipe_link10: mass 100.11 -> 0.0111
- link pipe_link11: mass 100.11 -> 0.0111
- link pipe_link12: mass 100.11 -> 0.0111
- link pipe_link13: mass 100.11 -> 0.0111
- link pipe_link14: mass 100.11 -> 0.0111
- link pipe_link15: mass 100.11 -> 0.0111
- link pipe_link17: mass 100.11 -> 0.0111
- link pipe_link18: mass 100.11 -> 0.0111
- link pipe_link19: mass 100.11 -> 0.0111
- link pipe_link2: mass 100.11 -> 0.0111
- link pipe_link20: mass 100.11 -> 0.0111
- link pipe_link21: mass 100.11 -> 0.0111
- link pipe_link22: mass 100.11 -> 0.0111
- link pipe_link23: mass 100.11 -> 0.0111
- link pipe_link24: mass 100.11 -> 0.0111
- link pipe_link3: mass 100.11 -> 0.0111
- link pipe_link4: mass 100.11 -> 0.0111
- link pipe_link5: mass 100.11 -> 0.0111
- link pipe_link6: mass 100.11 -> 0.0111
- link pipe_link7: mass 100.11 -> 0.0111
- link pipe_link8: mass 100.11 -> 0.0111
- link pipe_link9: mass 100.11 -> 0.0111
Joints:
- removed joint pipe_joint1100.11
- added joint pipe_joint10.0111: type continuous, parent pipe_link15, child pipe_link10.0111, origin xyz=0 5.5 0 rpy=0 0 0, axis 0 0 1, limit lower=-0.90.011171 upper=0.90.011171 effort=87 velocity=2.1750
- joint pipe_joint1: axis 1 0 0 -> (none); limit lower=-0.9100.1171 upper=0.9100.1171 effort=87 velocity=2.1750 -> (none); origin xyz=0 5.5 0 rpy=0 0 0 -> xyz=0 3 0 rpy=0 0 0; type continuous -> fixed
- joint pipe_joint10: limit lower=-0.9100.1171 upper=0.9100.1171 effort=87 velocity=2.1750 -> lower=-0.90.011171 upper=0.90.011171 effort=87 velocity=2.1750
- joint pipe_joint11: limit lower=-0.9100.1171 upper=0.9100.1171 effort=87 velocity=2.1750 -> lower=-0.90.011171 upper=0.90.011171 effort=87 velocity=2.1750
- joint pipe_joint12: limit lower=-0.9100.1171 upper=0.9100.1171 effort=87 velocity=2.1750 -> lower=-0.90.011171 upper=0.90.011171 effort=87 velocity=2.1750
- joint pipe_joint13: limit lower=-0.9100.1171 upper=0.9100.1171 effort=87 velocity=2.1750 -> lower=-0.90.011171 upper=0.90.011171 effort=87 velocity=2.1750
- joint pipe_joint14: limit lower=-0.9100.1171 upper=0.9100.1171 effort=87 velocity=2.1750 -> lower=-0.90.011171 upper=0.90.011171 effort=87 velocity=2.1750
- joint pipe_joint15: limit lower=-0.9100.1171 upper=0.9100.1171 effort=87 velocity=2.1750 -> lower=-0.90.011171 upper=0.90.011171 effort=87 velocity=2.1750
- joint pipe_joint17: limit lower=-0.9100.1171 upper=0.9100.1171 effort=87 velocity=2.1750 -> lower=-0.90.011171 upper=0.90.011171 effort=87 velocity=2.1750; parent pipe_link1100.11 -> pipe_link10.0111
- joint pipe_joint18: limit lower=-0.9100.1171 upper=0.9100.1171 effort=87 velocity=2.1750 -> lower=-0.90.011171 upper=0.90.011171 effort=87 velocity=2.1750
- joint pipe_joint19: limit lower=-0.9100.1171 upper=0.9100.1171 effort=87 velocity=2.1750 -> lower=-0.90.011171 upper=0.90.011171 effort=87 velocity=2.1750
- joint pipe_joint2: limit lower=-0.9100.1171 upper=0.9100.1171 effort=87 velocity=2.1750 -> lower=-0.90.011171 upper=0.90.011171 effort=87 velocity=2.1750
- joint pipe_joint20: limit lower=-0.9100.1171 upper=0.9100.1171 effort=87 velocity=2.1750 -> lower=-0.90.011171 upper=0.90.011171 effort=87 velocity=2.1750
- joint pipe_joint21: limit lower=-0.9100.1171 upper=0.9100.1171 effort=87 velocity=2.1750 -> lower=-0.90.011171 upper=0.90.011171 effort=87 velocity=2.1750
- joint pipe_joint22: limit lower=-0.9100.1171 upper=0.9100.1171 effort=87 velocity=2.1750 -> lower=-0.90.011171 upper=0.90.011171 effort=87 velocity=2.1750
- joint pipe_joint23: limit lower=-0.9100.1171 upper=0.9100.1171 effort=87 velocity=2.1750 -> lower=-0.90.011171 upper=0.90.011171 effort=87 velocity=2.1750
- joint pipe_joint24: limit lower=-0.9100.1171 upper=0.9100.1171 effort=87 velocity=2.1750 -> lower=-0.90.011171 upper=0.90.011171 effort=87 velocity=2.1750
- joint pipe_joint3: limit lower=-0.9100.1171 upper=0.9100.1171 effort=87 velocity=2.1750 -> lower=-0.90.011171 upper=0.90.011171 effort=87 velocity=2.1750
- joint pipe_joint4: limit lower=-0.9100.1171 upper=0.9100.1171 effort=87 velocity=2.1750 -> lower=-0.90.011171 upper=0.90.011171 effort=87 velocity=2.1750
- joint pipe_joint5: limit lower=-0.9100.1171 upper=0.9100.1171 effort=87 velocity=2.1750 -> lower=-0.90.011171 upper=0.90.011171 effort=87 velocity=2.1750
- joint pipe_joint6: limit lower=-0.9100.1171 upper=0.9100.1171 effort=87 velocity=2.1750 -> lower=-0.90.011171 upper=0.90.011171 effort=87 velocity=2.1750
- joint pipe_joint7: limit lower=-0.9100.1171 upper=0.9100.1171 effort=87 velocity=2.1750 -> lower=-0.90.011171 upper=0.90.011171 effort=87 velocity=2.1750
- joint pipe_joint8: limit lower=-0.9100.1171 upper=0.9100.1171 effort=87 velocity=2.1750 -> lower=-0.90.011171 upper=0.90.011171 effort=87 velocity=2.1750
- joint pipe_joint9: limit lower=-0.9100.1171 upper=0.9100.1171 effort=87 velocity=2.1750 -> lower=-0.90.011171 upper=0.90.011171 effort=87 velocity=2.1750
